File: electronics/motor_fader_main.kicad_sch (KiCad schematic)
At the start: 32 parts, among them J1 Conn_01x05, J2 Program, J3 Conn_01x05, J4 Conn_01x04_MountingPin, J5 Conn_01x04_MountingPin, U1 ATtiny1616-M, U2 DRV8837

Commit message: OMG update the MCU part number
Parts:
- U1: LCSC C2052778 -> C507118
Changed lines of the file:
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@@
 			)
 		)
-		(property "LCSC" "C2052778"
+		(property "LCSC" "C507118"
 			(at 54.61 88.9 0)
 			(effects
