File: electronics/fader_buddy_main.kicad_sch (KiCad schematic)
At the start: 32 parts, among them J1 Conn_01x05, J2 Program, J3 Conn_01x05, J4 Conn_01x04_MountingPin, J5 Conn_01x04_MountingPin, U1 ATtiny1616-M, U2 DRV8837

Commit message: schematic title block
Other:
- company: (none) -> https://github.com/scottbez1/FaderBuddy
- title: (none) -> FaderBuddy
Changed lines of the file:
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@@
 	(generator_version "10.0")
 	(paper "A4")
+	(title_block
+		(title "FaderBuddy")
+		(company "https://github.com/scottbez1/FaderBuddy")
+		(comment 1 "Apache 2.0 License")
+	)
 	(text "(Tx/Rx alt pins)"
 		(exclude_from_sim no)
