File: electronics/fader_buddy_main.kicad_sch (KiCad schematic)
At the start: 32 parts, among them J1 Conn_01x05, J2 Program, J3 Conn_01x05, J4 Conn_01x04_MountingPin, J5 Conn_01x04_MountingPin, U1 ATtiny1616-M, U2 DRV8837

Commit message: Update electronics to kicad 10 (#4)
Other:
- company: (none) -> https://github.com/scottbez1/FaderBuddy
- title: (none) -> FaderBuddy
